File: electronics/wolfgang_core/connectors.kicad_sch (KiCad schematic)
At the start: 0 parts

Commit message: Connectors copied
Parts:
- added HEAD1: BUS2_1, symbol Connector_Generic:Conn_01x04
- added JP1, JP2: M02, symbol Connector_Generic:Conn_01x02
- added LARM1: BUS3_1, symbol Connector_Generic:Conn_01x04
- added LLEG1: BUS0_1, symbol Connector_Generic:Conn_01x04
- added RARM1: BUS3_2, symbol Connector_Generic:Conn_01x04
- added RLEG1: BUS1_1, symbol Connector_Generic:Conn_01x04
Connections:
- new net +3.3V: JP1.2 (Pin_2), JP2.2 (Pin_2)
- new net GND: HEAD1.1 (Pin_1), JP1.1 (Pin_1), JP2.1 (Pin_1), LARM1.1 (Pin_1), LLEG1.1 (Pin_1), RARM1.1 (Pin_1), RLEG1.1 (Pin_1)
- new net VDXL: HEAD1.2 (Pin_2), LARM1.2 (Pin_2), LLEG1.2 (Pin_2), RARM1.2 (Pin_2), RLEG1.2 (Pin_2)
- new net dxl_0_n: LLEG1.3 (Pin_3)
- new net dxl_0_p: LLEG1.4 (Pin_4)
- new net dxl_1_n: RLEG1.3 (Pin_3)
- new net dxl_1_p: RLEG1.4 (Pin_4)
- new net dxl_2_n: HEAD1.3 (Pin_3)
- new net dxl_2_p: HEAD1.4 (Pin_4)
- new net dxl_3_n: LARM1.3 (Pin_3), RARM1.3 (Pin_3)
- new net dxl_3_p: LARM1.4 (Pin_4), RARM1.4 (Pin_4)

Commit message: Power largely done
Other:
- note added: "DXL Bus 0"
- note added: "DXL Bus 1"
- note added: "DXL Bus 2"
- note added: "DXL Bus 3"
- note added: "VCC Connectors"
Changed lines of the file:
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@@
     (stroke (width 0) (type default))
   )
-  (label "DXL Bus 3" (at 113.03 99.06 0) (fields_autoplaced)
+  (text "DXL Bus 3" (at 113.03 99.06 0)
     (effects (font (size 1.27 1.27)) (justify left bottom))
   )
-  (label "DXL Bus 1" (at 143.51 66.04 0) (fields_autoplaced)
+  (text "VCC Connectors\n" (at 151.13 110.49 0)
     (effects (font (size 1.27 1.27)) (justify left bottom))
   )
-  (label "DXL Bus 2" (at 175.26 66.04 0) (fields_autoplaced)
+  (text "DXL Bus 0" (at 113.03 66.04 0)
     (effects (font (size 1.27 1.27)) (justify left bottom))
   )
-  (label "VCC Connectors" (at 151.13 110.49 0) (fields_autoplaced)
+  (text "DXL Bus 2" (at 175.26 66.04 0)
     (effects (font (size 1.27 1.27)) (justify left bottom))
   )
-  (label "DXL Bus 0" (at 113.03 66.04 0) (fields_autoplaced)
+  (text "DXL Bus 1" (at 143.51 66.04 0)
     (effects (font (size 1.27 1.27)) (justify left bottom))
   )
@@
           (reference "LARM1") (unit 1)
         )
+        (path "/9538e4ed-27e6-4c37-b989-9859dc0d49e8/03085433-09a6-46e6-a151-340cb0e29306"
+          (reference "LARM2") (unit 1)
+        )
       )
     )
@@
           (reference "JP1") (unit 1)
         )
+        (path "/9538e4ed-27e6-4c37-b989-9859dc0d49e8/03085433-09a6-46e6-a151-340cb0e29306"
+          (reference "JP3") (unit 1)
+        )
       )
     )
@@
           (reference "JP2") (unit 1)
         )
+        (path "/9538e4ed-27e6-4c37-b989-9859dc0d49e8/03085433-09a6-46e6-a151-340cb0e29306"
+          (reference "JP4") (unit 1)
+        )
       )
     )
@@
           (reference "RLEG1") (unit 1)
         )
+        (path "/9538e4ed-27e6-4c37-b989-9859dc0d49e8/03085433-09a6-46e6-a151-340cb0e29306"
+          (reference "RLEG2") (unit 1)
+        )
       )
     )
@@
           (reference "#PWR010") (unit 1)
         )
+        (path "/9538e4ed-27e6-4c37-b989-9859dc0d49e8/03085433-09a6-46e6-a151-340cb0e29306"
+          (reference "#PWR018") (unit 1)
+        )
       )
     )
@@
           (reference "#PWR09") (unit 1)
         )
+        (path "/9538e4ed-27e6-4c37-b989-9859dc0d49e8/03085433-09a6-46e6-a151-340cb0e29306"
+          (reference "#PWR024") (unit 1)
+        )
       )
     )
@@
           (reference "#PWR014") (unit 1)
         )
+        (path "/9538e4ed-27e6-4c37-b989-9859dc0d49e8/03085433-09a6-46e6-a151-340cb0e29306"
+          (reference "#PWR022") (unit 1)
+        )
       )
     )
@@
           (reference "#PWR07") (unit 1)
         )
+        (path "/9538e4ed-27e6-4c37-b989-9859dc0d49e8/03085433-09a6-46e6-a151-340cb0e29306"
+          (reference "#PWR016") (unit 1)
+        )
       )
     )
@@
           (reference "LLEG1") (unit 1)
         )
+        (path "/9538e4ed-27e6-4c37-b989-9859dc0d49e8/03085433-09a6-46e6-a151-340cb0e29306"
+          (reference "LLEG2") (unit 1)
+        )
       )
     )
@@
           (reference "HEAD1") (unit 1)
         )
+        (path "/9538e4ed-27e6-4c37-b989-9859dc0d49e8/03085433-09a6-46e6-a151-340cb0e29306"
+          (reference "HEAD2") (unit 1)
+        )
       )
     )
@@
           (reference "#PWR08") (unit 1)
         )
+        (path "/9538e4ed-27e6-4c37-b989-9859dc0d49e8/03085433-09a6-46e6-a151-340cb0e29306"
+          (reference "#PWR019") (unit 1)
+        )
       )
     )
@@
           (reference "#PWR012") (unit 1)
         )
+        (path "/9538e4ed-27e6-4c37-b989-9859dc0d49e8/03085433-09a6-46e6-a151-340cb0e29306"
+          (reference "#PWR021") (unit 1)
+        )
       )
     )
@@
           (reference "#PWR013") (unit 1)
         )
+        (path "/9538e4ed-27e6-4c37-b989-9859dc0d49e8/03085433-09a6-46e6-a151-340cb0e29306"
+          (reference "#PWR020") (unit 1)
+        )
       )
     )
@@
           (reference "#PWR011") (unit 1)
         )
+        (path "/9538e4ed-27e6-4c37-b989-9859dc0d49e8/03085433-09a6-46e6-a151-340cb0e29306"
+          (reference "#PWR017") (unit 1)
+        )
       )
     )
@@
           (reference "#PWR015") (unit 1)
         )
+        (path "/9538e4ed-27e6-4c37-b989-9859dc0d49e8/03085433-09a6-46e6-a151-340cb0e29306"
+          (reference "#PWR023") (unit 1)
+        )
       )
     )
@@
           (reference "RARM1") (unit 1)
         )
-      )
+        (path "/9538e4ed-27e6-4c37-b989-9859dc0d49e8/03085433-09a6-46e6-a151-340cb0e29306"
+          (reference "RARM2") (unit 1)
+        )
+      )
