File: electronics/wolfgang_core/connectors.kicad_sch (KiCad schematic)
At the start: 7 parts

Commit message: Assign almost all Footprints
Parts:
- HEAD1, LARM1, LLEG1, RARM1, RLEG1: footprint (none) -> Connector_Molex:Molex_SPOX_5267-04A_1x04_P2.50mm_Vertical
- J1: renamed from JP1; footprint (none) -> Connector_Molex:Molex_SPOX_5267-02A_1x02_P2.50mm_Vertical
- J2: renamed from JP2; footprint (none) -> Connector_Molex:Molex_SPOX_5267-02A_1x02_P2.50mm_Vertical
Changed lines of the file:
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@@
 			)
 		)
-		(property "Footprint" ""
+		(property "Footprint" "Connector_Molex:Molex_SPOX_5267-04A_1x04_P2.50mm_Vertical"
 			(at 123.19 115.57 0)
 			(effects
@@
 		(dnp no)
 		(fields_autoplaced yes)
-		(property "Reference" "JP1"
+		(property "Reference" "J1"
 			(at 161.29 115.57 0)
 			(effects
@@
 			)
 		)
-		(property "Footprint" ""
+		(property "Footprint" "Connector_Molex:Molex_SPOX_5267-02A_1x02_P2.50mm_Vertical"
 			(at 161.29 124.46 0)
 			(effects
@@
 			(project "wolfgang_core"
 				(path "/9538e4ed-27e6-4c37-b989-9859dc0d49e8/ded4cb81-a8d4-43bd-a5d0-1be100709afa"
-					(reference "JP1")
+					(reference "J1")
 					(unit 1)
 				)
@@
 		(dnp no)
 		(fields_autoplaced yes)
-		(property "Reference" "JP2"
+		(property "Reference" "J2"
 			(at 176.53 115.57 0)
 			(effects
@@
 			)
 		)
-		(property "Footprint" ""
+		(property "Footprint" "Connector_Molex:Molex_SPOX_5267-02A_1x02_P2.50mm_Vertical"
 			(at 176.53 124.46 0)
 			(effects
@@
 			(project "wolfgang_core"
 				(path "/9538e4ed-27e6-4c37-b989-9859dc0d49e8/ded4cb81-a8d4-43bd-a5d0-1be100709afa"
-					(reference "JP2")
+					(reference "J2")
 					(unit 1)
 				)
@@
 			)
 		)
-		(property "Footprint" ""
+		(property "Footprint" "Connector_Molex:Molex_SPOX_5267-04A_1x04_P2.50mm_Vertical"
 			(at 153.67 82.55 0)
 			(effects
@@
 		(dnp no)
 		(fields_autoplaced yes)
-		(property "Reference" "#PWR029"
+		(property "Reference" "#PWR30"
 			(at 128.27 149.86 0)
 			(effects
@@
 			(project "wolfgang_core"
 				(path "/9538e4ed-27e6-4c37-b989-9859dc0d49e8/ded4cb81-a8d4-43bd-a5d0-1be100709afa"
-					(reference "#PWR029")
+					(reference "#PWR30")
 					(unit 1)
 				)
@@
 		(dnp no)
 		(fields_autoplaced yes)
-		(property "Reference" "#PWR035"
+		(property "Reference" "#PWR36"
 			(at 189.23 91.44 0)
 			(effects
@@
 			(project "wolfgang_core"
 				(path "/9538e4ed-27e6-4c37-b989-9859dc0d49e8/ded4cb81-a8d4-43bd-a5d0-1be100709afa"
-					(reference "#PWR035")
+					(reference "#PWR36")
 					(unit 1)
 				)
@@
 		(dnp no)
 		(fields_autoplaced yes)
-		(property "Reference" "#PWR033"
+		(property "Reference" "#PWR34"
 			(at 181.61 125.73 0)
 			(effects
@@
 			(project "wolfgang_core"
 				(path "/9538e4ed-27e6-4c37-b989-9859dc0d49e8/ded4cb81-a8d4-43bd-a5d0-1be100709afa"
-					(reference "#PWR033")
+					(reference "#PWR34")
 					(unit 1)
 				)
@@
 		(dnp no)
 		(fields_autoplaced yes)
-		(property "Reference" "#PWR027"
+		(property "Reference" "#PWR28"
 			(at 128.27 91.44 0)
 			(effects
@@
 			(project "wolfgang_core"
 				(path "/9538e4ed-27e6-4c37-b989-9859dc0d49e8/ded4cb81-a8d4-43bd-a5d0-1be100709afa"
-					(reference "#PWR027")
+					(reference "#PWR28")
 					(unit 1)
 				)
@@
 			)
 		)
-		(property "Footprint" ""
+		(property "Footprint" "Connector_Molex:Molex_SPOX_5267-04A_1x04_P2.50mm_Vertical"
 			(at 123.19 82.55 0)
 			(effects
@@
 			)
 		)
-		(property "Footprint" ""
+		(property "Footprint" "Connector_Molex:Molex_SPOX_5267-04A_1x04_P2.50mm_Vertical"
 			(at 184.15 82.55 0)
 			(effects
@@
 		(dnp no)
 		(fields_autoplaced yes)
-		(property "Reference" "#PWR030"
+		(property "Reference" "#PWR31"
 			(at 158.75 91.44 0)
 			(effects
@@
 			(project "wolfgang_core"
 				(path "/9538e4ed-27e6-4c37-b989-9859dc0d49e8/ded4cb81-a8d4-43bd-a5d0-1be100709afa"
-					(reference "#PWR030")
+					(reference "#PWR31")
 					(unit 1)
 				)
@@
 		(dnp no)
 		(fields_autoplaced yes)
-		(property "Reference" "#PWR032"
+		(property "Reference" "#PWR33"
 			(at 166.37 130.81 0)
 			(effects
@@
 			(project "wolfgang_core"
 				(path "/9538e4ed-27e6-4c37-b989-9859dc0d49e8/ded4cb81-a8d4-43bd-a5d0-1be100709afa"
-					(reference "#PWR032")
+					(reference "#PWR33")
 					(unit 1)
 				)
@@
 		(dnp no)
 		(fields_autoplaced yes)
-		(property "Reference" "#PWR031"
+		(property "Reference" "#PWR32"
 			(at 166.37 125.73 0)
 			(effects
@@
 			(project "wolfgang_core"
 				(path "/9538e4ed-27e6-4c37-b989-9859dc0d49e8/ded4cb81-a8d4-43bd-a5d0-1be100709afa"
-					(reference "#PWR031")
+					(reference "#PWR32")
 					(unit 1)
 				)
@@
 		(dnp no)
 		(fields_autoplaced yes)
-		(property "Reference" "#PWR028"
+		(property "Reference" "#PWR29"
 			(at 128.27 124.46 0)
 			(effects
@@
 			(project "wolfgang_core"
 				(path "/9538e4ed-27e6-4c37-b989-9859dc0d49e8/ded4cb81-a8d4-43bd-a5d0-1be100709afa"
-					(reference "#PWR028")
+					(reference "#PWR29")
 					(unit 1)
 				)
@@
 		(dnp no)
 		(fields_autoplaced yes)
-		(property "Reference" "#PWR034"
+		(property "Reference" "#PWR35"
 			(at 181.61 130.81 0)
 			(effects
@@
 			(project "wolfgang_core"
 				(path "/9538e4ed-27e6-4c37-b989-9859dc0d49e8/ded4cb81-a8d4-43bd-a5d0-1be100709afa"
-					(reference "#PWR034")
+					(reference "#PWR35")
 					(unit 1)
 				)
@@
 			)
 		)
-		(property "Footprint" ""
+		(property "Footprint" "Connector_Molex:Molex_SPOX_5267-04A_1x04_P2.50mm_Vertical"
 			(at 123.19 140.97 0)
 			(effects

Commit message: Fix Spox Stecker
Connections:
- net GND: now also HEAD1.4 (Pin_4), LARM1.4 (Pin_4), LLEG1.4 (Pin_4), RARM1.4 (Pin_4), RLEG1.4 (Pin_4); no longer HEAD1.1 (Pin_1), LARM1.1 (Pin_1), LLEG1.1 (Pin_1), RARM1.1 (Pin_1), RLEG1.1 (Pin_1)
- net VDXL: now also HEAD1.3 (Pin_3), LARM1.3 (Pin_3), LLEG1.3 (Pin_3), RARM1.3 (Pin_3), RLEG1.3 (Pin_3); no longer HEAD1.2 (Pin_2), LARM1.2 (Pin_2), LLEG1.2 (Pin_2), RARM1.2 (Pin_2), RLEG1.2 (Pin_2)
- net dxl_0_n: now also LLEG1.2 (Pin_2); no longer LLEG1.3 (Pin_3)
- net dxl_0_p: now also LLEG1.1 (Pin_1); no longer LLEG1.4 (Pin_4)
- net dxl_1_n: now also RLEG1.2 (Pin_2); no longer RLEG1.3 (Pin_3)
- net dxl_1_p: now also RLEG1.1 (Pin_1); no longer RLEG1.4 (Pin_4)
- net dxl_2_n: now also HEAD1.2 (Pin_2); no longer HEAD1.3 (Pin_3)
- net dxl_2_p: now also HEAD1.1 (Pin_1); no longer HEAD1.4 (Pin_4)
- net dxl_3_n: now also LARM1.2 (Pin_2), RARM1.2 (Pin_2); no longer LARM1.3 (Pin_3), RARM1.3 (Pin_3)
- net dxl_3_p: now also LARM1.1 (Pin_1), RARM1.1 (Pin_1); no longer LARM1.4 (Pin_4), RARM1.4 (Pin_4)
Other:
- moved on the sheet: HEAD1, LARM1, LLEG1, RARM1, RLEG1
Changed lines of the file:
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@@
 	(symbol
 		(lib_id "Connector_Generic:Conn_01x04")
-		(at 123.19 115.57 180)
-		(unit 1)
-		(exclude_from_sim no)
-		(in_bom yes)
-		(on_board yes)
-		(dnp no)
-		(fields_autoplaced yes)
+		(at 123.19 113.03 0)
+		(mirror y)
+		(unit 1)
+		(exclude_from_sim no)
+		(in_bom yes)
+		(on_board yes)
+		(dnp no)
 		(property "Reference" "LARM1"
-			(at 123.19 104.14 0)
+			(at 123.19 124.46 0)
 			(effects
 				(font
@@
 		)
 		(property "Value" "BUS3_1"
-			(at 123.19 106.68 0)
+			(at 123.19 121.92 0)
 			(effects
 				(font
@@
 		)
 		(property "Footprint" "Connector_Molex:Molex_SPOX_5267-04A_1x04_P2.50mm_Vertical"
-			(at 123.19 115.57 0)
+			(at 123.19 113.03 0)
 			(effects
 				(font
@@
 		)
 		(property "Datasheet" "~"
-			(at 123.19 115.57 0)
-			(effects
-				(font
-					(size 1.27 1.27)
-				)
-				(hide yes)
-			)
-		)
-		(property "Description" ""
-			(at 123.19 115.57 0)
+			(at 123.19 113.03 0)
+			(effects
+				(font
+					(size 1.27 1.27)
+				)
+				(hide yes)
+			)
+		)
+		(property "Description" ""
+			(at 123.19 113.03 0)
 			(effects
 				(font
@@
 	(symbol
 		(lib_id "Connector_Generic:Conn_01x04")
-		(at 153.67 82.55 180)
-		(unit 1)
-		(exclude_from_sim no)
-		(in_bom yes)
-		(on_board yes)
-		(dnp no)
-		(fields_autoplaced yes)
+		(at 153.67 80.01 0)
+		(mirror y)
+		(unit 1)
+		(exclude_from_sim no)
+		(in_bom yes)
+		(on_board yes)
+		(dnp no)
 		(property "Reference" "RLEG1"
-			(at 153.67 71.12 0)
+			(at 153.67 91.44 0)
 			(effects
 				(font
@@
 		)
 		(property "Value" "BUS1_1"
-			(at 153.67 73.66 0)
+			(at 153.67 88.9 0)
 			(effects
 				(font
@@
 		)
 		(property "Footprint" "Connector_Molex:Molex_SPOX_5267-04A_1x04_P2.50mm_Vertical"
-			(at 153.67 82.55 0)
+			(at 153.67 80.01 0)
 			(effects
 				(font
@@
 		)
 		(property "Datasheet" "~"
-			(at 153.67 82.55 0)
-			(effects
-				(font
-					(size 1.27 1.27)
-				)
-				(hide yes)
-			)
-		)
-		(property "Description" ""
-			(at 153.67 82.55 0)
+			(at 153.67 80.01 0)
+			(effects
+				(font
+					(size 1.27 1.27)
+				)
+				(hide yes)
+			)
+		)
+		(property "Description" ""
+			(at 153.67 80.01 0)
 			(effects
 				(font
@@
 	(symbol
 		(lib_id "Connector_Generic:Conn_01x04")
-		(at 123.19 82.55 180)
-		(unit 1)
-		(exclude_from_sim no)
-		(in_bom yes)
-		(on_board yes)
-		(dnp no)
-		(fields_autoplaced yes)
+		(at 123.19 80.01 0)
+		(mirror y)
+		(unit 1)
+		(exclude_from_sim no)
+		(in_bom yes)
+		(on_board yes)
+		(dnp no)
 		(property "Reference" "LLEG1"
-			(at 123.19 71.12 0)
+			(at 123.19 91.44 0)
 			(effects
 				(font
@@
 		)
 		(property "Value" "BUS0_1"
-			(at 123.19 73.66 0)
+			(at 123.19 88.9 0)
 			(effects
 				(font
@@
 		)
 		(property "Footprint" "Connector_Molex:Molex_SPOX_5267-04A_1x04_P2.50mm_Vertical"
-			(at 123.19 82.55 0)
+			(at 123.19 80.01 0)
 			(effects
 				(font
@@
 		)
 		(property "Datasheet" "~"
-			(at 123.19 82.55 0)
-			(effects
-				(font
-					(size 1.27 1.27)
-				)
-				(hide yes)
-			)
-		)
-		(property "Description" ""
-			(at 123.19 82.55 0)
+			(at 123.19 80.01 0)
+			(effects
+				(font
+					(size 1.27 1.27)
+				)
+				(hide yes)
+			)
+		)
+		(property "Description" ""
+			(at 123.19 80.01 0)
 			(effects
 				(font
@@
 	(symbol
 		(lib_id "Connector_Generic:Conn_01x04")
-		(at 184.15 82.55 180)
-		(unit 1)
-		(exclude_from_sim no)
-		(in_bom yes)
-		(on_board yes)
-		(dnp no)
-		(fields_autoplaced yes)
+		(at 184.15 80.01 0)
+		(mirror y)
+		(unit 1)
+		(exclude_from_sim no)
+		(in_bom yes)
+		(on_board yes)
+		(dnp no)
 		(property "Reference" "HEAD1"
-			(at 184.15 71.12 0)
+			(at 184.15 91.44 0)
 			(effects
 				(font
@@
 		)
 		(property "Value" "BUS2_1"
-			(at 184.15 73.66 0)
+			(at 184.15 88.9 0)
 			(effects
 				(font
@@
 		)
 		(property "Footprint" "Connector_Molex:Molex_SPOX_5267-04A_1x04_P2.50mm_Vertical"
-			(at 184.15 82.55 0)
+			(at 184.15 80.01 0)
 			(effects
 				(font
@@
 		)
 		(property "Datasheet" "~"
-			(at 184.15 82.55 0)
-			(effects
-				(font
-					(size 1.27 1.27)
-				)
-				(hide yes)
-			)
-		)
-		(property "Description" ""
-			(at 184.15 82.55 0)
+			(at 184.15 80.01 0)
+			(effects
+				(font
+					(size 1.27 1.27)
+				)
+				(hide yes)
+			)
+		)
+		(property "Description" ""
+			(at 184.15 80.01 0)
 			(effects
 				(font
@@
 	(symbol
 		(lib_id "Connector_Generic:Conn_01x04")
-		(at 123.19 140.97 180)
-		(unit 1)
-		(exclude_from_sim no)
-		(in_bom yes)
-		(on_board yes)
-		(dnp no)
-		(fields_autoplaced yes)
+		(at 123.19 138.43 0)
+		(mirror y)
+		(unit 1)
+		(exclude_from_sim no)
+		(in_bom yes)
+		(on_board yes)
+		(dnp no)
 		(property "Reference" "RARM1"
-			(at 123.19 129.54 0)
+			(at 123.19 149.86 0)
 			(effects
 				(font
@@
 		)
 		(property "Value" "BUS3_2"
-			(at 123.19 132.08 0)
+			(at 123.19 147.32 0)
 			(effects
 				(font
@@
 		)
 		(property "Footprint" "Connector_Molex:Molex_SPOX_5267-04A_1x04_P2.50mm_Vertical"
-			(at 123.19 140.97 0)
+			(at 123.19 138.43 0)
 			(effects
 				(font
@@
 		)
 		(property "Datasheet" "~"
-			(at 123.19 140.97 0)
-			(effects
-				(font
-					(size 1.27 1.27)
-				)
-				(hide yes)
-			)
-		)
-		(property "Description" ""
-			(at 123.19 140.97 0)
-			(effects
-				(font
+			(at 123.19 138.43 0)
+			(effects
+				(font
+					(size 1.27 1.27)
+				)
+				(hide yes)
+			)
+		)
+		(property "Description" ""
+			(at 123.19 138.43 0)
+			(effects
+				(font
